Commit message: More playing with HARLIE in gazebo

File: cwru_semi_stable/cwru_urdf/harlie.urdf.xacro (robot description, xacro)
@@ -1,7 +1,8 @@
 <?xml version="1.0"?>
-<robot xmlns:sensor="http://playerstage.sourceforge.net/gazebo/xmlschema/#sensor"
-	 xmlns:controller="http://playerstage.sourceforge.net/gazebo/xmlschema/#controller"
-	 xmlns:interface="http://playerstage.sourceforge.net/gazebo/xmlschema/#interface"
-	 xmlns:xacro="http://playerstage.sourceforge.net/gazebo/xmlschema/#interface" name="macroed">
+<robot  xmlns:sensor="http://playerstage.sourceforge.net/gazebo/xmlschema/#sensor"
+	xmlns:controller="http://playerstage.sourceforge.net/gazebo/xmlschema/#controller"
+	xmlns:interface="http://playerstage.sourceforge.net/gazebo/xmlschema/#interface"
+	xmlns:xacro="http://playerstage.sourceforge.net/gazebo/xmlschema/#interface"
+	name="harlie">
 	<include filename="$(find cwru_urdf)/sensors/sick_lms291_laser.urdf.xacro" />
 	<xacro:property name="bodylen" value="0.5461" />
@@ -39,8 +40,8 @@
 	<xacro:macro name="default_inertial" params="mass">
 		<inertial>
-      			<mass value="${mass}" />
-		        <inertia ixx="1.0" ixy="0.0" ixz="0.0"
-			         iyy="1.0" iyz="0.0"
-			         izz="1.0" />
+			<mass value="${mass}" />
+			<inertia ixx="1.0" ixy="0.0" ixz="0.0"
+				iyy="1.0" iyz="0.0"
+				izz="1.0" />
 		</inertial>
 	</xacro:macro>
@@ -67,5 +68,5 @@
 			<child link="${prefix}_wheel"/>
 			<origin xyz="0 ${reflect*track/2} ${wheeldrop}" rpy="0 ${M_PI/2} ${M_PI/2}"/>
-      			<limit effort="100" velocity="100" />
+			<limit effort="100" velocity="100" />
 			<joint_properties damping="0.0" friction="0.0" />
 		</joint>
@@ -187,5 +188,5 @@
 			<child link="${prefix}_casterwheel"/>
 			<origin xyz="${-casterwidth/2-.02} .053 -.053" rpy="0 ${M_PI/2} 0"/>
-      			<limit effort="100" velocity="100" />
+			<limit effort="100" velocity="100" />
 			<joint_properties damping="0.0" friction="0.0" />
 		</joint>
@@ -209,5 +210,10 @@
 			<origin xyz="${originX} ${originY} ${originZ}" rpy="0 0 0"/>
 		</collision>
-		<xacro:default_inertial mass="1"/>
+		<inertial>
+			<mass value="158.75" />
+			<inertia ixx="5.5" ixy="-0.0097199" ixz="1.293988"
+				iyy="5.5" iyz="-0.0073"
+				izz="3.7" />
+		</inertial>
 	</link>
 	<link name="mastleft">
@@ -257,5 +263,5 @@
 		<origin xyz="${bodylen/2+originX-boschwidth/2} ${-bodywidth/2+boschwidth/2} ${mastheight/2-bodyheight/2+originZ}" />
 	</joint>
-		<link name="masttop">
+	<link name="masttop">
 		<visual>
 			<geometry>
@@ -298,5 +304,5 @@
 			<origin xyz="0 0 0" rpy="0 0 0"/>
 		</collision>
-		<xacro:default_inertial mass="30"/>
+		<xacro:default_inertial mass="1"/>
 	</link>
 	<joint name="batterytobase" type="fixed">

Commit message: More improvements to HARLIE gazebo simulation

File: cwru_semi_stable/cwru_urdf/harlie.urdf.xacro (robot description, xacro)
@@ -41,7 +41,7 @@
 		<inertial>
 			<mass value="${mass}" />
-			<inertia ixx="1.0" ixy="0.0" ixz="0.0"
-				iyy="1.0" iyz="0.0"
-				izz="1.0" />
+			<inertia ixx="0.01" ixy="0.001" ixz="0.001"
+				iyy="0.01" iyz="0.001"
+				izz="0.01" />
 		</inertial>
 	</xacro:macro>
