Commit message: Started adding SICK LIDAR to urdf.
Defining a macro for a SICK LMS291 in the cwru_description package.
Still need to figure out some transforms.

File: cwru_semi_stable/cwru_description/urdf/gazebo.urdf.xacro (robot description, xacro)
@@ -27,3 +27,28 @@
   </gazebo>
 </xacro:macro>
+<xacro:macro name="sim_sick_lidar">
+  <gazebo reference="laser_scan_link">
+    <sensor:ray name="laser_scan_link">
+     <rayCount>181</rayCount>
+     <rangeCount>181</rangeCount>
+     <laserCount>1</laserCount>
+         <origin>0.0 0.0 0.0</origin>
+         <displayRays>true</displayRays>
+         <minAngle>-90</minAngle>
+         <maxAngle>90</maxAngle>
+         <minRange>0.06</minRange>
+         <maxRange>30.0</maxRange>
+         <resRange>0.01</resRange>
+         <updateRate>10.0</updateRate>
+         <controller:gazebo_ros_laser name="gazebo_ros_base_scan_link_controller" plugin="libgazebo_ros_laser.so">
+                <gaussianNoise>0.005</gaussianNoise>
+                <alwaysOn>true</alwaysOn>
+                <updateRate>20.0</updateRate>
+                <topicName>base_scan/scan</topicName>
+                <frameName>laser_scan_link</frameName>
+                <interface:laser name="gazebo_ros_base_scan_link_iface"/>
+         </controller:gazebo_ros_laser>
+        </sensor:ray>
+  </gazebo>
+</xacro:macro>
 </robot>
