Commit message: Finished sick LIDAR xacro.
The LIDAR is now loaded into the model with a xacro in the cwru_description.
The xacro macro includes the model and the tf for the LIDAR, which allows
the removal of the tf broadcaster from the launch file.

File: cwru_semi_stable/cwru_description/urdf/sick_LMS291.urdf.xacro (robot description, xacro)
@@ -3,6 +3,6 @@
   <property name="M_PI" value="3.14159"/>
   <include filename="$(find cwru_description)/urdf/gazebo.urdf.xacro"/>
-<xacro:macro name="SICK_LMS291" params="xyz rpy parent_frame" >
-	<joint name="base_camera_joint" type="fixed">
+<xacro:macro name="SICK_LMS291" params="xyz rpy parent_frame laser_frame" >
+  <joint name="base_laser_joint" type="fixed">
     <origin xyz="${xyz}" rpy="${rpy}" />
     <parent link="${parent_frame}" />
@@ -13,5 +13,5 @@
 		<visual>
 			<geometry>
-				<mesh filename="package://cwru_description/meshes/sick lms291.stl" scale="0.0254 0.0254 0.0254"/>
+				<mesh filename="package://cwru_description/meshes/sick_lms291.stl" scale="0.0254 0.0254 0.0254"/>
 			</geometry>
 			<origin rpy="0 0 0" xyz="-0.0683999139953 -0.00245779587475 -0.0929987962566"/>
@@ -27,10 +27,10 @@
 		<collision>
 			<geometry>
-				<mesh filename="package://cwru_description/meshes/sick lms291.stl" scale="0.0254 0.0254 0.0254"/>
+				<mesh filename="package://cwru_description/meshes/sick_lms291.stl" scale="0.0254 0.0254 0.0254"/>
 			</geometry>
 			<origin rpy="0 0 0" xyz="-0.0683999139953 -0.00245779587475 -0.0929987962566"/>
 		</collision>
 	</link>
-  <link name="SICK_laser_frame">
+  <link name="${laser_frame}">
     <inertial>
       <mass value="0.01" />
@@ -42,7 +42,7 @@
   </link>
   <joint name="SICK_laser_frame_joint" type="fixed">
-    <origin xyz="0 0 0" rpy="${-M_PI/2} 0 ${-M_PI/2}" />
-    <parent link="camera_depth_frame" />
-    <child link="camera_depth_optical_frame" />
+    <origin xyz="-0.0683999139953 0.035 -0.093" rpy="1.266 1.571 2.837" />
+    <parent link="SICK_LMS291" />
+    <child link="${laser_frame}" />
   </joint>
 </xacro:macro>

Commit message: Fixes LIDAR definition and adds self filter.
LIDAR definition had the sensor frame off by about 6cm.
Also fixes abby's Kinect to match the corrected LIDAR frame.
Also adds self-filtering to the arm launch file.

File: cwru_semi_stable/cwru_description/urdf/sick_LMS291.urdf.xacro (robot description, xacro)
@@ -42,5 +42,5 @@
   </link>
   <joint name="SICK_laser_frame_joint" type="fixed">
-    <origin xyz="-0.0683999139953 0.035 -0.093" rpy="1.266 1.571 2.837" />
+    <origin xyz="-0.0683999139953 0.035 -0.0273" rpy="1.266 1.571 2.837" />
     <parent link="SICK_LMS291" />
     <child link="${laser_frame}" />
