Commit message: Updated kinect macro.
Kinect optical frames are published by the camera driver, making the
optical frames in the URDF redundant. Moved these to a separate macro.

File: cwru_semi_stable/cwru_description/urdf/kinect.urdf.xacro (robot description, xacro)
@@ -31,4 +31,6 @@
     </collision>
   </link>
+</xacro:macro>
+<xacro:macro name="kinect_frames">
   <joint name="camera_depth_joint" type="fixed">
     <origin xyz="0 0.018 0" rpy="0 0 0" />

Commit message: Fixed kinect and arm frames.
Kinect now publishes frames for rgb and depth in the correct
place. (curse you willowgarage).

IRB-120 has been moved and rotated to reflect the fact that the rail it is
mounted to is not actually vertical. A more complete fix would be to rotate
the whole frame in the model to be correct, but this will do for now.

File: cwru_semi_stable/cwru_description/urdf/kinect.urdf.xacro (robot description, xacro)
@@ -31,8 +31,6 @@
     </collision>
   </link>
-</xacro:macro>
-<xacro:macro name="kinect_frames">
   <joint name="camera_depth_joint" type="fixed">
-    <origin xyz="0 0.018 0" rpy="0 0 0" />
+    <origin xyz="0 0.011 0" rpy="0 0 0" />
     <parent link="camera_link" />
     <child link="camera_depth_frame" />
@@ -62,5 +60,5 @@
   </link>
   <joint name="camera_rgb_joint" type="fixed">
-    <origin xyz="0 -0.005 0" rpy="0 0 0" />
+    <origin xyz="0 -0.012 0" rpy="0 0 0" />
     <parent link="camera_link" />
     <child link="camera_rgb_frame" />
