Commit message: robot interface and corresponding abby gazebo modeo w/ control

File: catkin/src/cwru_376_student/abby_wsn_dev/rrbot_description/urdf/rrbot.xacro (robot description, xacro)
@@ -59,5 +59,5 @@
     <child link="link2"/>
     <origin xyz="0 0 0.0" rpy="0 0 0"/>
-    <limit effort="10" lower="-2.87979" upper="2.87979" velocity="4.36332"/>
+    <limit effort="100" lower="-2.87979" upper="2.87979" velocity="4.36332"/>
     <axis xyz="0 0 1"/>
     <dynamics damping="0.7"/>
@@ -93,5 +93,5 @@
     <origin rpy="0 0 0" xyz="0 0 0.29"/>
     <axis xyz="0 1 0"/>
-    <limit effort="10" lower="-1.91986" upper="1.91986" velocity="4.36332"/>
+    <limit effort="100" lower="-1.91986" upper="1.91986" velocity="4.36332"/>
     <dynamics damping="1.7"/>
   </joint>
@@ -150,5 +150,5 @@
     <origin rpy="0 0 0" xyz="0 0 0.27"/>
     <axis xyz="0 1 0"/>
-   <limit effort="10" lower="-1.91986" upper="1.22173" velocity="4.36332"/>
+   <limit effort="100" lower="-1.91986" upper="1.22173" velocity="4.36332"/>
     <dynamics damping="1.7"/>
   </joint>
@@ -182,5 +182,5 @@
     <origin rpy="0 0 0" xyz="0 0 0.07"/>
     <axis xyz="1 0 0"/>
-    <limit effort="10" lower="-2.79253" upper="2.79253" velocity="5.58505"/>
+    <limit effort="20" lower="-2.79253" upper="2.79253" velocity="5.58505"/>
     <dynamics damping="1.7"/>
   </joint>
@@ -214,5 +214,5 @@
    <origin rpy="0 0 0" xyz="0.302 0 0"/>
     <axis xyz="0 1 0"/>
-     <limit effort="10" lower="-2.094395" upper="2.094395" velocity="5.58505"/>
+     <limit effort="20" lower="-2.094395" upper="2.094395" velocity="5.58505"/>
     <dynamics damping="1.7"/>
   </joint>
@@ -246,5 +246,5 @@
     <origin rpy="0 0 0" xyz="0.072 0 0"/>
     <axis xyz="1 0 0"/>
-     <limit effort="10" lower="-6.98132" upper="6.98132" velocity="7.33038"/>
+     <limit effort="20" lower="-6.98132" upper="6.98132" velocity="7.33038"/>
     <dynamics damping="0.7"/>
   </joint>
@@ -309,3 +309,8 @@
     </actuator>
   </transmission>
+<gazebo>
+  <plugin name="gazebo_ros_control" filename="libgazebo_ros_control.so">
+    <robotNamespace>/rrbot</robotNamespace>
+  </plugin>
+</gazebo>
 </robot>
